File: dimmer.kicad_sch (KiCad schematic)
At the start: 53 parts, among them J1 Screw_Terminal_01x07, J2 Screw_Terminal_01x02, J3 KNX-IN, J4 Screw_Terminal_01x08, Q1 2N2222A, Q10 2N2222A, Q11 2N2222A, Q12 IRFZ44N, Q13 2N2222A, Q14 2N2222A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

Commit message: Cleanup Schematics
Parts:
- added C1: 0.1μF, Capacitor_THT:CP_Radial_D4.0mm_P1.50mm, symbol Device:C
Connections:
- net +5V: now also C1.1
- net GND: now also C1.2
Other:
- moved on the sheet: H2, H3, H4, J1, J2, J3, J4, JP1, U1
