File: _autosave-dimmer.kicad_sch (KiCad schematic)
At the start: 54 parts, among them J1 Screw_Terminal_01x07, J2 Screw_Terminal_01x02, J3 KNX-IN, J4 Screw_Terminal_01x08, Q1 2N2222A, Q10 2N2222A, Q11 2N2222A, Q12 IRFZ44N, Q13 2N2222A, Q14 2N2222A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

Commit message: div cleanups
Connections:
- net +12V: now also J1.7 (Pin_7); no longer J1.1 (Pin_1)
- net +3.3V: now also J4.2 (Pin_2); no longer J4.7 (Pin_7)
- net GND: now also J4.1 (Pin_1); no longer J4.8 (Pin_8)
- net GPIO_IN1: now also J4.3 (Pin_3); no longer J4.6 (Pin_6)
- net GPIO_IN2: now also J4.4 (Pin_4); no longer J4.5 (Pin_5)
- net GPIO_IN3: now also J4.5 (Pin_5); no longer J4.4 (Pin_4)
- net GPIO_IN4: now also J4.6 (Pin_6); no longer J4.3 (Pin_3)
- net GPIO_IN5: now also J4.7 (Pin_7); no longer J4.2 (Pin_2)
- net GPIO_IN6: now also J4.8 (Pin_8); no longer J4.1 (Pin_1)
- net LED1: now also J1.1 (Pin_1); no longer J1.7 (Pin_7)
- net LED2: now also J1.2 (Pin_2); no longer J1.6 (Pin_6)
- net LED3: now also J1.3 (Pin_4); no longer J1.5 (Pin_5)
- net LED5: now also J1.5 (Pin_5); no longer J1.3 (Pin_3)
- net LED6: now also J1.6 (Pin_6); no longer J1.2 (Pin_2)
Changed lines of the file:
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@@
       (effects (font (size 1.27 1.27)) hide)
     )
-    (pin "1")
-    (pin "2")
-    (pin "3")
+    (pin "8")
+    (pin "7")
+    (pin "6")
+    (pin "5")
     (pin "4")
-    (pin "5")
-    (pin "6")
-    (pin "7")
-    (pin "8")
+    (pin "3")
+    (pin "2")
+    (pin "1")
     (instances
       (project "dimmer"
@@
       (effects (font (size 1.27 1.27)) hide)
     )
-    (pin "1")
-    (pin "2")
-    (pin "3")
+    (pin "7")
+    (pin "6")
+    (pin "5")
     (pin "4")
-    (pin "5")
-    (pin "6")
-    (pin "7")
-    (instances
-      (project "dimmer"
+    (pin "3")
+    (pin "2")
+    (pin "1")
+    (instances
+      (project "dimmer"
