File: dimmer.kicad_pcb (KiCad board)
At the start: 2 copper layers, 160 x 100 mm, 53 parts, among them J1 Screw_Terminal_01x07, J2 Screw_Terminal_01x02, J3 KNX-IN, J4 Screw_Terminal_01x08, Q1 2N2222A, Q10 2N2222A, Q11 2N2222A, Q12 IRFZ44N, Q13 2N2222A, Q14 2N2222A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

Commit message: div changes
Parts:
- added C1: 0.1μF, Capacitor_THT:CP_Radial_D4.0mm_P1.50mm, F.Cu at (31.5, 77.0)
- moved U1 5.92 mm to (25.0, 82.0)
Routing:
- net +5V: track 268.9 -> 281.4 mm
- net +12V: track 45.7 -> 44.6 mm

Commit message: div cleanups
Parts:
- moved J4 35.0 mm to (111.0, 110.0), turned to 0 degrees
- moved J1 30.0 mm to (30.0, 33.0), turned to -90 degrees
- moved JP1 13.3 mm to (156.0, 112.5), turned to 180 degrees
- moved J3 6.96 mm to (83.5, 85.0)
- moved Q14 1.00 mm to (140.0, 32.0)
Connections:
- J1 pad 1: +12V -> /LED1
- J1 pad 2: /LED6 -> /LED2
- J1 pad 3: /LED5 -> /LED3
- J1 pad 5: /LED3 -> /LED5
- J1 pad 6: /LED2 -> /LED6
- J1 pad 7: /LED1 -> +12V
- J4 pad 1: /GPIO_IN6 -> GND
- J4 pad 2: /GPIO_IN5 -> +3.3V
- J4 pad 3: /GPIO_IN4 -> /GPIO_IN1
- J4 pad 4: /GPIO_IN3 -> /GPIO_IN2
- J4 pad 5: /GPIO_IN2 -> /GPIO_IN3
- J4 pad 6: /GPIO_IN1 -> /GPIO_IN4
- J4 pad 7: +3.3V -> /GPIO_IN5
- J4 pad 8: GND -> /GPIO_IN6
- JP1 pad 1: +5V -> KNX +5V
- JP1 pad 3: KNX +5V -> +5V
- Q12 pad 1: /LED4 -> Net-(Q11-C)
- Q12 pad 2: Net-(Q11-C) -> /LED4
- Q15 pad 1: /LED5 -> Net-(Q14-C)
- Q15 pad 2: Net-(Q14-C) -> /LED5
- Q18 pad 1: /LED6 -> Net-(Q17-C)
- Q18 pad 2: Net-(Q17-C) -> /LED6
- Q3 pad 1: /LED1 -> Net-(Q2-C)
- Q3 pad 2: Net-(Q2-C) -> /LED1
- Q6 pad 1: /LED2 -> Net-(Q5-C)
- Q6 pad 2: Net-(Q5-C) -> /LED2
- Q9 pad 1: /LED3 -> Net-(Q8-C)
- Q9 pad 2: Net-(Q8-C) -> /LED3
Routing:
- net /ESP +5v IN: track 13.6 -> 27.2 mm
- net KNX +5V: track 99.8 -> 88.3 mm
- net +5V: track 281.4 -> 290.1 mm
- net /RXD: track 87.5 -> 89.6 mm
- net Net-(Q13-C): track 11.4 -> 10.4 mm
- net Net-(Q14-C): track 17.7 -> 18.3 mm

Commit message: div updates
Parts:
- added C2: 0.1μF 25V, Capacitor_THT:CP_Radial_D18.0mm_P7.50mm, F.Cu at (35.0, 100.0)
- moved JP1 135.0 mm to (23.5, 86.5)
- moved C1 36.2 mm to (35.3, 113.0), turned to 0 degrees
- moved J2 31.0 mm to (30.0, 75.0)
- moved U1 24.6 mm to (24.5, 106.6)
- moved J3 9.81 mm to (93.0, 82.4)
- moved Q15 9.00 mm to (128.5, 24.9)
- moved Q18 8.80 mm to (149.7, 24.8)
- moved Q12 7.26 mm to (107.7, 24.8)
- moved Q17 6.62 mm to (154.8, 32.3)
- moved Q16 6.13 mm to (155.1, 38.2)
- moved R21 6.13 mm to (153.9, 43.2)
- moved R22 6.13 mm to (158.9, 43.2)
- moved R23 6.13 mm to (148.9, 51.5)
- moved R24 6.13 mm to (143.9, 51.5)
- moved Q13 6.11 mm to (134.2, 37.7)
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Connections:
- JP1 pad 1: KNX +5V -> KNX +20V
- JP1 pad 2: /ESP +5v IN -> /Regulator_IN
- JP1 pad 3: +5V -> +12V
- U1 pad 1: +12V -> /Regulator_IN
Routing:
- net KNX +5V: track 88.3 -> 0.00 mm
- net KNX +20V: track 0.00 -> 69.9 mm
- net /Regulator_IN: track 0.00 -> 38.9 mm
- net /ESP +5v IN: track 27.2 -> 0.00 mm
- net +12V: track 44.6 -> 21.1 mm
- net /TXD: track 86.0 -> 73.9 mm
- net /RXD: track 89.6 -> 78.5 mm
- net +5V: track 290.1 -> 301.1 mm
- net /LED6: track 152.8 -> 144.7 mm
- net /LED5: track 129.2 -> 122.5 mm
- net /LED4: track 99.8 -> 93.8 mm
- net /LED1: track 27.6 -> 22.3 mm
- net /LED5_GPIO: track 21.1 -> 25.8 mm
- net /LED4_GPIO: track 40.1 -> 44.8 mm
- net Net-(Q14-C): track 18.3 -> 14.0 mm
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Other:
- board text added: "Kanal 1"
- board text added: "Kanal 2"
- board text added: "Kanal 3"
- board text added: "Kanal 4"
- board text added: "Kanal 5"
- board text added: "Kanal 6"
